File: Tutorial PCB/Tutorial PCB.kicad_pcb (KiCad board)
At the start: 2 copper layers, 71.4 x 38.1 mm, 24 parts, among them SW1 SW_Push, U1 ATmega32U4-A, Y1 16MHz

Commit message: 1
Routing:
- net +5V: track 27.6 -> 60.4 mm, vias 0 -> 2
- net GND: track 79.3 -> 105.1 mm, vias 0 -> 2
Changed lines of the file:
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@@
 		(at 40.48125 25.675 -90)
 		(property "Reference" "USB1"
-			(at -0.9 0 180)
+			(at -0.9 0 0)
 			(layer "B.CrtYd")
 			(effects
@@
 		)
 		(property "Value" "Molex-0548190519"
-			(at -5.08 0 180)
+			(at -5.08 0 0)
 			(layer "Dwgs.User")
 			(effects
@@
 		)
 		(fp_text user "${REFERENCE}"
-			(at 2.45 0 180)
+			(at 2.45 0 0)
 			(layer "B.SilkS")
 			(effects
@@
 	)
 	(segment
+		(start 43.65625 50.02175)
+		(end 43.65625 48.53125)
+		(width 0.381)
+		(layer "F.Cu")
+		(net 1)
+	)
+	(via
+		(at 43.65625 48.53125)
+		(size 0.6)
+		(drill 0.3)
+		(layers "F.Cu" "B.Cu")
+		(net 1)
+	)
+	(via
+		(at 43.65625 50.02175)
+		(size 0.6)
+		(drill 0.3)
+		(layers "F.Cu" "B.Cu")
+		(net 1)
+	)
+	(segment
 		(start 51.369875 38.2125)
 		(end 53.069875 36.5125)
@@
 	)
 	(segment
+		(start 41.24375 58.23125)
+		(end 41.24375 60.14375)
+		(width 0.381)
+		(layer "B.Cu")
+		(net 1)
+	)
+	(segment
 		(start 51.175 60.325)
 		(end 47.625 60.325)
@@
 	)
 	(segment
+		(start 43.41275 48.53125)
+		(end 43.65625 48.53125)
+		(width 0.381)
+		(layer "B.Cu")
+		(net 1)
+	)
+	(segment
 		(start 53.31875 58.18125)
 		(end 51.175 60.325)
@@
 	)
 	(segment
+		(start 43.65625 48.53125)
+		(end 50.14375 48.53125)
+		(width 0.381)
+		(layer "B.Cu")
+		(net 1)
+	)
+	(segment
 		(start 47.625 60.325)
 		(end 43.0125 60.325)
@@
 	)
 	(segment
+		(start 43.65625 52.325)
+		(end 43.65625 50.02175)
+		(width 0.381)
+		(layer "B.Cu")
+		(net 1)
+	)
+	(segment
 		(start 57.277875 37.47275)
 		(end 57.277875 40.680125)
@@
 	)
 	(segment
+		(start 41.24375 54.7375)
+		(end 41.24375 58.23125)
+		(width 0.381)
+		(layer "B.Cu")
+		(net 1)
+	)
+	(segment
 		(start 56.51025 41.44775)
 		(end 56.51025 45.9835)
@@
 	)
 	(segment
+		(start 41.24375 54.7375)
+		(end 43.65625 52.325)
+		(width 0.381)
+		(layer "B.Cu")
+		(net 1)
+	)
+	(segment
 		(start 34.125 55.06875)
 		(end 35.8625 53.33125)
@@
 	)
 	(segment
+		(start 38.74375 53.33125)
+		(end 39.8375 53.33125)
+		(width 0.381)
+		(layer "B.Cu")
+		(net 1)
+	)
+	(segment
 		(start 43.0125 43.00625)
 		(end 42.84375 43.175)
@@
 	)
 	(segment
+		(start 42.84375 46.83125)
+		(end 42.84375 47.96225)
+		(width 0.381)
+		(layer "B.Cu")
+		(net 1)
+	)
+	(segment
+		(start 41.24375 60.14375)
+		(end 42.21875 61.11875)
+		(width 0.381)
+		(layer "B.Cu")
+		(net 1)
+	)
+	(segment
+		(start 42.84375 47.96225)
+		(end 43.41275 48.53125)
+		(width 0.381)
+		(layer "B.Cu")
+		(net 1)
+	)
+	(segment
 		(start 32.975062 53.918812)
 		(end 34.125 55.06875)
@@
 		(start 56.005125 36.5125)
 		(end 56.161375 36.35625)
+		(width 0.381)
+		(layer "B.Cu")
+		(net 1)
+	)
+	(segment
+		(start 39.8375 53.33125)
+		(end 41.24375 54.7375)
 		(width 0.381)
 		(layer "B.Cu")
@@
 	)
 	(segment
+		(start 40.572633 56.171367)
+		(end 40.44375 56.30025)
+		(width 0.381)
+		(layer "F.Cu")
+		(net 3)
+	)
+	(segment
+		(start 40.572633 53.089867)
+		(end 40.572633 56.171367)
+		(width 0.381)
+		(layer "F.Cu")
+		(net 3)
+	)
+	(via
+		(at 40.572633 53.089867)
+		(size 0.6)
+		(drill 0.3)
+		(layers "F.Cu" "B.Cu")
+		(net 3)
+	)
+	(via
+		(at 40.44375 56.30025)
+		(size 0.6)
+		(drill 0.3)
+		(layers "F.Cu" "B.Cu")
+		(net 3)
+	)
+	(segment
+		(start 39.87475 55.73125)
+		(end 38.74375 55.73125)
+		(width 0.381)
+		(layer "B.Cu")
+		(net 3)
+	)
+	(segment
+		(start 48.41875 49.33125)
+		(end 42.27475 49.33125)
+		(width 0.381)
+		(layer "B.Cu")
+		(net 3)
+	)
+	(segment
+		(start 39.87475 51.73125)
+		(end 38.74375 51.73125)
+		(width 0.381)
+		(layer "B.Cu")
+		(net 3)
+	)
+	(segment
 		(start 41.1125 43.00625)
 		(end 42.04375 43.9375)
@@
 	)
 	(segment
+		(start 42.27475 49.33125)
+		(end 42.04375 49.56225)
+		(width 0.381)
+		(layer "B.Cu")
+		(net 3)
+	)
+	(segment
 		(start 37.45 43.00625)
 		(end 41.1125 43.00625)
@@
 	)
 	(segment
+		(start 42.04375 49.56225)
+		(end 39.87475 51.73125)
+		(width 0.381)
+		(layer "B.Cu")
+		(net 3)
+	)
+	(segment
+		(start 39.87475 51.73125)
+		(end 40.572633 52.429133)
+		(width 0.381)
+		(layer "B.Cu")
+		(net 3)
+	)
+	(segment
+		(start 40.44375 56.30025)
+		(end 39.87475 55.73125)
+		(width 0.381)
+		(layer "B.Cu")
+		(net 3)
+	)
+	(segment
 		(start 37.30625 42.8625)
 		(end 37.45 43.00625)
@@
 	)
 	(segment
+		(start 40.44375 58.23125)
+		(end 40.44375 56.30025)
+		(width 0.381)
+		(layer "B.Cu")
+		(net 3)
+	)
+	(segment
 		(start 54.1125 50.28125)
 		(end 53.1625 49.33125)
@@
 	)
 	(segment
+		(start 50.14375 49.33125)
+		(end 48.41875 49.33125)
+		(width 0.381)
+		(layer "B.Cu")
+		(net 3)
+	)
+	(segment
+		(start 40.572633 52.429133)
+		(end 40.572633 53.089867)
+		(width 0.381)
+		(layer "B.Cu")
+		(net 3)
+	)
+	(segment
 		(start 36.98125 42.8625)
 		(end 37.30625 42.8625)
@@
 	)
 	(segment
+		(start 42.04375 46.83125)
+		(end 42.04375 49.56225)
+		(width 0.381)
+		(layer "B.Cu")
+		(net 3)
+	)
+	(segment
 		(start 40.96875 42.8625)
 		(end 41.1125 43.00625)
@@
 		(width 0.381)
 		(layer "B.Cu")
+		(net 3)
+	)
+	(segment
+		(start 48.44375 49.35625)
+		(end 48.41875 49.33125)
+		(width 0.381)
+		(layer "B.Cu")
+		(net 3)
+	)
+	(segment
+		(start 48.44375 58.23125)
+		(end 48.44375 49.35625)
+		(width 0.381)
+		(layer "B.Cu")
